File: Electrique/SoM_V1/SoM_ESP32_v1/Communication.kicad_sch (KiCad schematic)
At the start: 4 parts, among them U301 TCA9546APWR, U302 MCP2515-xST, U303 FT231XS

Commit message: push pcb
Parts:
- added C301, C305, C309, C310: 0.1µF, Resistor_SMD:R_0805_2012Metric, symbol Device:C
- added C302, C303: 47pF, Resistor_SMD:R_0805_2012Metric, symbol Device:C
- added C304, C308: 10µF, Resistor_SMD:R_0805_2012Metric, symbol Device:C
- added C306, C307: 22pF, Resistor_SMD:R_0805_2012Metric, symbol Device:C
- added D309: TX, LED_SMD:LED_0805_2012Metric, symbol Device:LED
- added D310: RX, LED_SMD:LED_0805_2012Metric, symbol Device:LED
- added R301, R302: 27, Resistor_SMD:R_0805_2012Metric, symbol Device:R_US
- added R303, R304, R305, R306, R307, R308, R309, R310, R311, R312, R313: 1k, Resistor_SMD:R_0805_2012Metric, symbol Device:R_US
- added R314, R315: 330, Resistor_SMD:R_0805_2012Metric, symbol Device:R_US
- added R316: 10k, Resistor_SMD:R_0805_2012Metric, symbol Device:R_US
- added U304: TJA1051T, Package_SO:SOIC-8_3.9x4.9mm_P1.27mm, symbol Interface_CAN_LIN:TJA1051T
- added Y301: 8MHz, Crystal:Crystal_SMD_Abracon_ABM3-2Pin_5.0x3.2mm, symbol Device:Crystal
- U301: footprint PW0016A-IPC_A -> Package_SO:TSSOP-16_4.4x5mm_P0.65mm
Connections:
- net DTR: now reaches U303.1 (~{DTR})
- net D+: now reaches U303.11 (USBDP)
- net D+: now also R302.2
- net D-: now reaches U303.12 (USBDM)
- net D-: now also R301.2
- net Vcc_3V3: now reaches U303.13 (3V3OUT)
- net Vcc_3V3: now also U301.16 (VCC), U302.20 (VDD), U303.14 (~{RESET}), U303.15 (VCC), U303.3 (VCCIO), C301.1, C304.1, C305.1, C308.1, C309.1, C310.1, R303.1, R304.1, R305.1, R306.1, R307.1, R308.1, R309.1, R310.1, R311.1, R312.1, R313.1, R314.2, R315.2, R316.1, U304.3 (VCC)
- net GND: now reaches U303.16 (GND)
- net GND: now also U301.1 (A0), U301.13 (A2), U301.2 (A1), U301.8 (GND), U302.10 (VSS), U303.6 (GND), C301.2, C302.2, C303.2, C304.2, C305.2, C306.2, C307.2, C308.2, C309.2, C310.2, U304.2 (GND), U304.8 (S)
- net RTS: now reaches U303.2 (~{RTS})
- net U0RXD: now reaches U303.20 (TXD)
- net U0RXD: now also D309.1 (K)
- net U0TXD: now reaches U303.4 (RXD)
- net U0TXD: now also D310.1 (K)
- net GPIO17_U1_TXD: now reaches J201.22 (UART_TX)
- net GPIO18_U1_RXD: now reaches J201.32 (UART_RX)
- net at J201.71 (CAN_H_MCP2515): now also U304.7 (CANH)
- net at J201.73 (CAN_L_MCP2515): now also U304.6 (CANL)
- net DEBUG-: now reaches J201.46 (USB_DEBUG_D-)
- net DEBUG+: now reaches J201.48 (USB_DEBUG_D+)
- net at U302.1 (TXCAN): now also U304.1 (TXD)
- net GPIO48/CAN_INT: now reaches U302.13 (~{INT})
- net SPI_CLK_ESP32: now reaches U302.14 (SCK)
- net SPI_CLK_ESP32: now also J201.23 (SPI_CLK)
- net SPI_MOSI_ESP32: now reaches U302.16 (SI)
- net SPI_MOSI_ESP32: now also J201.35 (SPI_MOSI)
- net SPI_MISO_ESP32: now reaches U302.17 (SO)
- net SPI_MISO_ESP32: now also J201.37 (SPI_MISO)
- net SPI_CAN_ESP32: now reaches U302.18 (~{CS})
- net RESET_OTHERS: now reaches U302.19 (~{RESET})
- net RESET_OTHERS: now also U301.3 (RESET_N), R313.2, R316.2
- net at U302.2 (RXCAN): now also U304.4 (RXD)
- net at U302.8 (OSC2): now also C306.1, Y301.2
- net at U302.9 (OSC1): now also C307.1, Y301.1
- net I2C_SCL_0_TCA: now reaches J201.11 (I2C_SCL_1_TCA)
- net I2C_SCL_0_TCA: now also U301.5 (SC0), R311.2
- net I2C_SDA_1_TCA: now reaches J201.13 (I2C_SDA_2_TCA)
- net I2C_SDA_1_TCA: now also U301.6 (SD1), R306.2
- net I2C_SDA_2_TCA: now reaches J201.14 (I2C_SDA_3_TCA)
- net I2C_SDA_2_TCA: now also U301.9 (SD2), R309.2
- net I2C_SCL_1_TCA: now reaches J201.15 (I2C_SCL_2_TCA)
- net I2C_SCL_1_TCA: now also U301.7 (SC1), R312.2
- net I2C_SCL_2_TCA: now reaches J201.16 (I2C_SCL_3_TCA)
- net I2C_SCL_2_TCA: now also U301.10 (SC2), R310.2
- net I2C_SDA_3_TCA: now reaches J201.17 (I2C_SDA_4_TCA)
- net I2C_SDA_3_TCA: now also U301.11 (SD3), R307.2
- net I2C_SCL_3_TCA: now reaches J201.19 (I2C_SCL_4_TCA)
- net I2C_SCL_3_TCA: now also U301.12 (SC3), R308.2
- net I2C_SDA_ESP32: now reaches J201.58 (I2C_SDA_ESP32)
- net I2C_SDA_ESP32: now also U301.15 (SDA), R303.2
- net I2C_SCL_ESP32: now reaches J201.60 (I2C_SCL_ESP32)
- net I2C_SCL_ESP32: now also U301.14 (SCL), R304.2
- net I2C_SDA_0_TCA: now reaches J201.9 (I2C_SDA_1_TCA)
- net I2C_SDA_0_TCA: now also U301.4 (SD0), R305.2
- net DR+: now reaches J201.3 (USB_D+_FT231)
- net DR+: now also C303.1, R302.1
- net DR-: now reaches J201.5 (USB_D-_FT231)
- net DR-: now also C302.1, R301.1
- net SPI_5_ESP32: now reaches J201.20 (SPI_CS_5)
- net SPI_6_ESP32: now reaches J201.21 (SPI_CS_6)
- net I2S_WS: now reaches J201.10 (I2S_WS)
- net I2S_DIN/DOUT: now reaches J201.12 (I2S_DIN/DOUT)
- net I2S_BCLK: now reaches J201.8 (I2S_BCLK)
- new net: D309.2 (A), R314.1
- new net: D310.2 (A), R315.1
- no-connect marks 0 -> 14
Other:
- note added: "ABM3-8.000MHZ-B4Y-T"
- moved on the sheet: J201B, J201C, J201D, J201E, J201F, J201G, J201H, U301, U302, U303
