File: Electrique/SoM_V1/SoM_ESP32_v1/ESP32.kicad_sch (KiCad schematic)
At the start: 1 part, among them U701 ESP32-S3-WROOM-2

Commit message: push pcb
Parts:
- added C601, C605: 0.1µF, Resistor_SMD:R_0805_2012Metric, symbol Device:C_Small
- added C602, C606: 1µF, Resistor_SMD:R_0805_2012Metric, symbol Device:C
- added C603: 10µF, Resistor_SMD:R_0805_2012Metric, symbol Device:C
- added C604, C607: 0.1µF, Resistor_SMD:R_0805_2012Metric, symbol Device:C
- added Q603: MBT3904DW1T1G, Package_TO_SOT_SMD:SOT-363_SC-70-6, symbol Transistor_BJT:UMH3N
- added R601, R602, R605, R606, R607: 10k, Resistor_SMD:R_0805_2012Metric, symbol Device:R_US
- added SW601: SW_BOOT, Button_Switch_SMD:SW_DIP_SPSTx01_Slide_6.7x4.1mm_W6.73mm_P2.54mm_LowProfile_JPin, symbol Switch:SW_Push
- added SW602: SW_CHIP_EN, Button_Switch_SMD:SW_DIP_SPSTx01_Slide_6.7x4.1mm_W6.73mm_P2.54mm_LowProfile_JPin, symbol Switch:SW_Push
- added U601: 74HC238, Package_SO:SOIC-16_3.9x9.9mm_P1.27mm, symbol 74xx:74HC238
Connections:
- net GND: now reaches U701.1 (GND), U701.40 (GND), U701.41 (GND)
- net GND: now also C601.2, C602.2, C603.2, C604.2, C605.2, C606.2, C607.2, R601.2, R602.2, SW601.2, SW602.2, U601.8 (GND)
- net GPIO17_U1_TXD: now reaches U701.10 (IO17)
- net GPIO18_U1_RXD: now reaches U701.11 (IO18)
- net SPI_MISO_ESP32: now reaches U701.12 (IO8)
- net DEBUG-: now reaches U701.13 (USB_D-/IO19)
- net DEBUG+: now reaches U701.14 (USB_D+/IO20)
- net at U701.16 (IO46): now also R602.1
- net REFCLKn: now reaches U701.17 (IO9)
- net SUSCLK: now reaches U701.18 (IO10)
- net RESET_OTHERS: now reaches U701.19 (IO11)
- net Vcc_3V3: now reaches U701.2 (3V3)
- net Vcc_3V3: now also C603.1, C604.1, C606.1, C607.1, R607.1, U601.16 (VCC), U601.6 (E3)
- net I2S_BCLK: now reaches U701.20 (IO12)
- net I2S_WS: now reaches U701.21 (IO13)
- net I2S_DIN/DOUT: now reaches U701.22 (IO14)
- net at U701.23 (IO21): now also U601.3 (A2)
- net GPIO47: now reaches U701.24 (IO47)
- net GPIO48/CAN_INT: now reaches U701.25 (IO48)
- net at U701.26 (IO45): now also R601.1
- net GPIO0_BOOT: now reaches U701.27 (IO0)
- net GPIO0_BOOT: now also C601.1, Q603.4 (E2), SW601.1
- net CHIP_EN: now reaches U701.3 (EN)
- net CHIP_EN: now also C602.1, C605.1, Q603.6 (C1), R607.2, SW602.1
- net GPIO38_ADDRESSABLE_LED: now reaches U701.31 (IO38)
- net U0RXD: now reaches U701.36 (RXD0/IO44)
- net U0TXD: now reaches U701.37 (TXD0/IO43)
- net I2C_SCL_ESP32: now reaches U701.38 (IO2)
- net I2C_SDA_ESP32: now reaches U701.39 (IO1)
- net at U701.4 (IO4): now also U601.1 (A0)
- net at U701.5 (IO5): now also U601.2 (A1)
- net SPI_CLK_ESP32: now reaches U701.6 (IO6)
- net SPI_MOSI_ESP32: now reaches U701.7 (IO7)
- net GPIO15: now reaches U701.8 (IO15)
- net GPIO16: now reaches U701.9 (IO16)
- new net: Q603.2 (B1), R605.2
- new net: Q603.5 (B2), R606.2
- new net DTR: Q603.3 (C2), R605.1
- new net LDAC_DAC: U601.11 (Y4)
- new net RTS: Q603.1 (E1), R606.1
- new net SPI_5_ESP32: U601.10 (Y5)
- new net SPI_6_ESP32: U601.9 (Y6)
- new net SPI_7_ESP32: U601.7 (Y7)
- new net SPI_ADC_ESP32: U601.13 (Y2)
- new net SPI_CAN_ESP32: U601.15 (Y0)
- new net SPI_DAC_ESP32: U601.12 (Y3)
- new net SPI_SD_ESP32: U601.14 (Y1)
- no-connect marks 0 -> 7
Other:
- note added: "Auto program: DTR RTS --> EN BOOT GPIO2 1 1 1 1 1 0 0 1 1 1 1 0 0 1 1 0 1 1 0 0"
