File: Electrique/SoM_V1/SoM_ESP32_v1/Sortie.kicad_sch (KiCad schematic)
At the start: 2 parts, among them U501 PCA9633DP1

Commit message: push pcb
Parts:
- added C501: 1µF, Resistor_SMD:R_0805_2012Metric, symbol Device:C
- added C502: 100nF, Resistor_SMD:R_0805_2012Metric, symbol Device:C
- added C503: 100n, Capacitor_SMD:C_0805_2012Metric, symbol Device:C
- added D501: FZ2812-5050, LED_SMD:LED_Inolux_IN-PI554FCH_PLCC4_5.0x5.0mm_P3.2mm, symbol LED:Inolux_IN-PI554FCH
- added R501, R502: 10k, Resistor_SMD:R_0805_2012Metric, symbol Device:R_US
Connections:
- net at J201.64 (PWM_1_PCA): now also U501.1 (PWM1)
- net at J201.66 (PWM_2_PCA): now also U501.2 (SCL6)
- net at J201.68 (PWM_3_PCA): now also U501.3 (PWM3)
- net at J201.70 (PWM_4_PCA): now also U501.4 (PWM4)
- net GPIO47: now reaches J201.34 (GPIO47)
- net GPIO48/CAN_INT: now reaches J201.36 (GPIO48)
- net GPIO15: now reaches J201.40 (GPIO15)
- net GPIO16: now reaches J201.41 (GPIO16)
- net GPIO38_ADDRESSABLE_LED: now reaches J201.6 (GPIO38&LED)
- net GPIO38_ADDRESSABLE_LED: now also D501.2 (DIN)
- net I2C_SCL_ESP32: now reaches U501.2 (SCL6)
- net I2C_SCL_ESP32: now also R502.2
- net GND: now reaches U501.5 (GND)
- net GND: now also C501.2, C502.2, C503.2, D501.1 (VSS)
- net I2C_SDA_ESP32: now reaches U501.7 (SDA)
- net I2C_SDA_ESP32: now also R501.2
- net Vcc_3V3: now reaches U501.8 (VCC)
- net Vcc_3V3: now also C501.1, C502.1, C503.1, D501.3 (VDD), R501.1, R502.1
- net SUSCLK: now reaches J201.50 (SUSCLK)
- no-connect marks 0 -> 8
Other:
- note added: "ERREUR ICI dans la V1: pin SDA et SCL n'était pas bien nommé. Erreur réglé pour la V2."
- note added: "REFCLK n'est pas un feature En gros le SDK de ESP-IDF ne le supporte pas???? https://www.esp32.com/viewtopic.php?t=3011 à vérifier"
- moved on the sheet: J201J, J201K, J201L, U501
