File: Electrique/MOBO_V1/MOBO_V1/MOBO_V1.kicad_sch (KiCad schematic)
At the start: 1 part

Commit message: Push de 3 nouveau board/PCB
Parts:
- J101: footprint (none) -> MDT320E01001:AMPHENOL_MDT320E01001
Connections:
- net SUSCLK: now reaches J101.50 (SUSCLK)
- net SPI_5_ESP32: now reaches J101.20 (SPI_CS_5)
- net SPI_6_ESP32: now reaches J101.21 (SPI_CS_6)
- net SPI_CLK_ESP32: now reaches J101.23 (SPI_CLK)
- net SPI_MOSI_ESP32: now reaches J101.35 (SPI_MOSI)
- net SPI_MISO_ESP32: now reaches J101.37 (SPI_MISO)
- net FT231_D+: now reaches J101.3 (USB_D+_FT231)
- net FT231_D-: now reaches J101.5 (USB_D-_FT231)
- net DAC_1: now reaches J101.59 (DAC_1_MCP48)
- net DAC_2: now reaches J101.61 (DAC_2_MCP48)
- net ADC_1: now reaches J101.65 (ADC_1_MCP3202)
- net ADC_2: now reaches J101.67 (ADC_2_MCP3202)
- net GPIO47: now reaches J101.34 (GPIO47)
- net GPIO48/CAN_INT: now reaches J101.36 (GPIO48)
- net GPIO15: now reaches J101.40 (GPIO15)
- net GPIO16: now reaches J101.41 (GPIO16)
- net GPIO26: now reaches J101.42 (GPIO26)
- net GPIO33: now reaches J101.43 (GPIO33)
- net GPIO34: now reaches J101.44 (GPIO34)
- net GPIO45: now reaches J101.52 (GPIO45)
- net GPIO46: now reaches J101.53 (GPIO46)
- net GPIO38_ADDRESSABLE_LED: now reaches J101.6 (GPIO38&LED)
- net CAN_H: now reaches J101.71 (CAN_H_MCP2515)
- net CAN_L: now reaches J101.73 (CAN_L_MCP2515)
- net I2C_SCL_0_TCA: now reaches J101.11 (I2C_SCL_1_TCA)
- net I2C_SDA_1_TCA: now reaches J101.13 (I2C_SDA_2_TCA)
- net I2C_SDA_2_TCA: now reaches J101.14 (I2C_SDA_3_TCA)
- net I2C_SCL_1_TCA: now reaches J101.15 (I2C_SCL_2_TCA)
- net I2C_SCL_2_TCA: now reaches J101.16 (I2C_SCL_3_TCA)
- net I2C_SDA_3_TCA: now reaches J101.17 (I2C_SDA_4_TCA)
- net I2C_SCL_3_TCA: now reaches J101.19 (I2C_SCL_4_TCA)
- net I2C_SDA_ESP32: now reaches J101.58 (I2C_SDA_ESP32)
- net I2C_SCL_ESP32: now reaches J101.60 (I2C_SCL_ESP32)
- net I2C_SDA_0_TCA: now reaches J101.9 (I2C_SDA_1_TCA)
- net I2S_WS: now reaches J101.10 (I2S_WS)
- net I2S_DIN/DOUT: now reaches J101.12 (I2S_DIN/DOUT)
- net I2S_BCLK: now reaches J101.8 (I2S_BCLK)
- net GPIO17_U1_TXD: now reaches J101.22 (UART_TX)
- net GPIO18_U1_RXD: now reaches J101.32 (UART_RX)
- net GND: now reaches J101.1 (GND)
- net GND: now also J101.18 (GND), J101.33 (GND), J101.38 (GND), J101.39 (GND), J101.45 (GND), J101.51 (GND), J101.55 (GND), J101.57 (GND), J101.62 (GND), J101.63 (GND), J101.69 (GND), J101.7 (GND), J101.75 (GND)
- net Vcc_3V3: now reaches J101.2 (Vcc_3v3)
- net Vcc_3V3: now also J101.4 (Vcc_3v3), J101.72 (Vcc_3v3), J101.74 (Vcc_3v3)
- net RESET_OTHERS: now reaches J101.54 (RESET_AUTRES)
- net CHIP_EN: now reaches J101.56 (RESET_ESP32)
- net PWM_1: now reaches J101.64 (PWM_1_PCA)
- net PWM_2: now reaches J101.66 (PWM_2_PCA)
- net PWM_3: now reaches J101.68 (PWM_3_PCA)
- net PWM_4: now reaches J101.70 (PWM_4_PCA)
- net DEBUG_D-: now reaches J101.46 (USB_DEBUG_D-)
- net DEBUG_D+: now reaches J101.48 (USB_DEBUG_D+)
- no-connect marks 0 -> 2
Other:
- added sheet connexion (connexion.kicad_sch)
- added sheet power (power.kicad_sch)
