File: Electrique/SoM_V2/SoM_V2/SoM_V2.kicad_sch (KiCad schematic)
At the start: 0 parts

Commit message: push fix ???
Other:
- removed sheet Analogue
Changed lines of the file:
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@@
 	(paper "A4")
 	(sheet
-		(at 215.9 15.24)
-		(size 68.58 142.24)
+		(at 115.57 90.17)
+		(size 98.425 68.58)
 		(fields_autoplaced yes)
 		(stroke
@@
 		)
 		(property "Sheetname" "ESP32"
-			(at 215.9 14.5284 0)
+			(at 115.57 89.4584 0)
 			(effects
 				(font
@@
 		)
 		(property "Sheetfile" "ESP32.kicad_sch"
-			(at 215.9 158.0646 0)
+			(at 115.57 159.3346 0)
 			(effects
 				(font
@@
 	)
 	(sheet
-		(at 13.97 88.9)
-		(size 99.06 68.58)
-		(fields_autoplaced yes)
-		(stroke
-			(width 0.1524)
-			(type solid)
-		)
-		(fill
-			(color 0 0 0 0.0000)
-		)
-		(property "Sheetname" "Analogue"
-			(at 13.97 88.1884 0)
-			(effects
-				(font
-					(size 1.27 1.27)
-				)
-				(justify left bottom)
-			)
-		)
-		(property "Sheetfile" "Analogue.kicad_sch"
-			(at 13.97 158.0646 0)
-			(effects
-				(font
-					(size 1.27 1.27)
-				)
-				(justify left top)
-			)
-		)
-		(instances
-			(project "SoM_V2"
-				(path "/ecd44d9a-8113-48e2-a5bb-0de07ce8b9ce"
-					(page "4")
-				)
-			)
-		)
-	)
-	(sheet
 		(at 13.97 15.24)
 		(size 99.06 68.58)
@@
 	)
 	(sheet
-		(at 115.57 88.9)
+		(at 13.97 90.17)
 		(size 99.06 68.58)
 		(fields_autoplaced yes)
@@
 		)
 		(property "Sheetname" "Sortie"
-			(at 115.57 88.1884 0)
+			(at 13.97 89.4584 0)
 			(effects
 				(font
@@
 		)
 		(property "Sheetfile" "Sortie.kicad_sch"
-			(at 115.57 158.0646 0)
+			(at 13.97 159.3346 0)
 			(effects
 				(font
