File: Electrique/SoM_V2/SoM_V2/Communication.kicad_sch (KiCad schematic)
At the start: 27 parts, among them U301 TCA9546APWR, U302 MCP2515-xST, U303 TJA1051T, U304 FT231XS, Y301 8MHz

Commit message: stinky kicad
Connections:
- net DR+: now also J201.3 (USB_D+_FT231); no longer J201.5 (USB_D+_FT231)
- net DR-: now also J201.5 (USB_D-_FT231); no longer J201.3 (USB_D-_FT231)
Changed lines of the file:
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@@
 	)
 	(symbol
-		(lib_name "connecteur_SOM_ESP32_4")
 		(lib_id "connecteur_m2_key_E:connecteur_SOM_ESP32")
 		(at 228.6 91.44 0)
@@
 		(dnp no)
 		(property "Reference" "J201"
-			(at 228.6 85.09 0)
+			(at 227.838 88.138 0)
 			(effects
 				(font
@@
 		(dnp no)
 		(property "Reference" "J201"
-			(at 143.51 132.08 0)
+			(at 143.002 134.874 0)
 			(effects
 				(font
@@
 	)
 	(symbol
-		(lib_name "connecteur_SOM_ESP32_5")
 		(lib_id "connecteur_m2_key_E:connecteur_SOM_ESP32")
 		(at 237.49 100.33 0)
@@
 		(dnp no)
 		(property "Reference" "J201"
-			(at 237.49 93.98 0)
+			(at 236.982 97.028 0)
 			(effects
 				(font
@@
 	)
 	(symbol
-		(lib_name "connecteur_SOM_ESP32_1")
 		(lib_id "connecteur_m2_key_E:connecteur_SOM_ESP32")
 		(at 66.04 29.21 0)
@@
 	)
 	(symbol
-		(lib_name "connecteur_SOM_ESP32_2")
 		(lib_id "connecteur_m2_key_E:connecteur_SOM_ESP32")
 		(at 161.29 130.81 0)
@@
 		(on_board yes)
 		(dnp no)
-		(fields_autoplaced yes)
 		(property "Reference" "J201"
-			(at 161.29 124.46 0)
+			(at 161.036 126.492 0)
 			(effects
 				(font
@@
 	)
 	(symbol
-		(lib_name "connecteur_SOM_ESP32_3")
 		(lib_id "connecteur_m2_key_E:connecteur_SOM_ESP32")
 		(at 182.88 93.98 0)
@@
 		(on_board yes)
 		(dnp no)
-		(fields_autoplaced yes)
 		(property "Reference" "J201"
-			(at 182.88 87.63 0)
+			(at 184.15 86.36 0)
 			(effects
 				(font
@@
 	)
 	(symbol
-		(lib_name "connecteur_SOM_ESP32_6")
 		(lib_id "connecteur_m2_key_E:connecteur_SOM_ESP32")
 		(at 233.68 83.82 0)

Commit message: push fix ???
Parts:
- removed J201: ~, connecteur_M2_key_E:NGFF_E, symbol connecteur_m2_key_E:connecteur_SOM_ESP32
- added U201: ~, connecteur_M2_key_E:NGFF_E, symbol connecteur_m2_key_E:connecteur_SOM_ESP32_V2
- renumbered R309 to R305, R310 to R306, R313 to R307, R316 to R308
Connections:
- net DEBUG+: now also U201.3 (USB_D+_FT231)
- net DEBUG-: now also U201.5 (USB_D-_FT231)
- net DR+: now also U201.48 (USB_DEBUG_D+)
- net DR-: now also U201.46 (USB_DEBUG_D-)
- net GPIO17_U1_TXD: now also U201.22 (UART_TX)
- net GPIO18_U1_RXD: now also U201.32 (UART_RX)
- net I2C_SCL_0_TCA: now also U201.11 (I2C_SCL_1_TCA)
- net I2C_SCL_1_TCA: now also U201.15 (I2C_SCL_2_TCA)
- net I2C_SCL_2_TCA: now also U201.16 (I2C_SCL_3_TCA)
- net I2C_SCL_3_TCA: now also U201.19 (I2C_SCL_4_TCA)
- net I2C_SCL_ESP32: now also U201.60 (I2C_SCL_ESP32)
- net I2C_SDA_0_TCA: now also U201.9 (I2C_SDA_1_TCA)
- net I2C_SDA_1_TCA: now also U201.13 (I2C_SDA_2_TCA)
- net I2C_SDA_2_TCA: now also U201.14 (I2C_SDA_3_TCA)
- net I2C_SDA_3_TCA: now also U201.17 (I2C_SDA_4_TCA)
- net I2C_SDA_ESP32: now also U201.58 (I2C_SDA_ESP32)
- net I2S_BCLK: now also U201.8 (I2S_BCLK)
- net I2S_DIN/DOUT: now also U201.12 (I2S_DIN/DOUT)
- net I2S_WS: now also U201.10 (I2S_WS)
- net SPI_CLK_ESP32: now also U201.23 (SPI_CLK)
- net SPI_MISO_ESP32: now also U201.37 (SPI_MISO)
- net SPI_MOSI_ESP32: now also U201.35 (SPI_MOSI)
- net Vcc_3V3: now also U303.5 (V_{IO}); no longer U303.3 (VCC)
- net at U303.6 (CANL): now also U201.73 (CAN_L_MCP2515)
- net at U303.7 (CANH): now also U201.71 (CAN_H_MCP2515)
- new net CS_1: U201.20 (CS_1)
- new net CS_2: U201.21 (CS_2)
- new net Vcc_5V: U303.3 (Vcc_5V)

Commit message: push v2.2
Parts:
- removed U302: MCP2515-xST, Package_SO:TSSOP-20_4.4x6.5mm_P0.65mm, symbol Interface_CAN_LIN:MCP2515-xST
- removed U303: TJA1051T, Package_SO:SOIC-8_3.9x4.9mm_P1.27mm, symbol Interface_CAN_LIN:TJA1051T
- removed U304: FT231XS, Package_SO:SSOP-20_3.9x8.7mm_P0.635mm, symbol Interface_USB:FT231XS
- removed Y301: 8MHz, Crystal:Crystal_SMD_Abracon_ABM3-2Pin_5.0x3.2mm, symbol Device:Crystal
- added D303: SP0502BAJT, Package_TO_SOT_SMD:SOT-323_SC-70, symbol Power_Protection:SP0502BAJT
- added R309, R310: 1k, Resistor_SMD:R_0805_2012Metric, symbol Device:R_US
- added R311, R312: 60, Resistor_SMD:R_0805_2012Metric, symbol Device:R_US
- added U302: FT231XQ, Package_DFN_QFN:QFN-20-1EP_4x4mm_P0.5mm_EP2.5x2.5mm, symbol Interface_USB:FT231XQ
- added U305: SN65HVD230, Package_SO:SOIC-8_3.9x4.9mm_P1.27mm, symbol Interface_CAN_LIN:SN65HVD230
- C303: value 22pF -> 1µF
- C304: value 22pF -> 0.1µF
- C305: value 10µF -> 1µF
- R304: value 10k -> 1k
Connections:
- net D+: now also U302.8 (USBDP)
- net D-: now also U302.9 (USBDM)
- net DEBUG+: now also U201.48 (USB_DEBUG_D+); no longer U201.3 (USB_D+_FT231)
- net DEBUG-: now also U201.46 (USB_DEBUG_D-); no longer U201.5 (USB_D-_FT231)
- net DR+: now also U201.3 (USB_D+_FT231); no longer U201.48 (USB_DEBUG_D+)
- net DR-: now also U201.5 (USB_D-_FT231); no longer U201.46 (USB_DEBUG_D-)
- net DTR: now also U302.18 (~{DTR})
- net GND: now also C307.1, R310.1, U302.13 (GND), U302.21 (GND), U302.3 (GND), U305.2 (GND); no longer C303.2, C307.2
- net RESET_OTHERS: no longer R304.2
- net RTS: now also U302.19 (~{RTS})
- net U0RXD: now also U302.17 (TXD)
- net U0TXD: now also U302.1 (RXD)
- net Vcc_3V3: now also U302.10 (3V3OUT), U302.11 (~{RESET}), U302.12 (VCC), U302.20 (VCCIO), U305.3 (VCC); no longer C307.1, R304.1
- net CAN-: now reaches U201.73 (CAN_L_MCP2515)
- net CAN-: now also C304.1, D303.2 (K), R312.2, U305.6 (CANL)
- net CAN+: now reaches U201.71 (CAN_H_MCP2515)
- net CAN+: now also C307.2, D303.1 (K), R311.1, U305.7 (CANH)
- net Vref_CAN: now reaches C303.1
- net Vref_CAN: now also R311.2, R312.1, U305.5 (Vref)
- new net: R309.2, U305.4 (R)
- new net: C303.2, D303.3 (A)
- new net: R304.2, U305.1 (D)
- new net: R310.2, U305.8 (Rs)
- new net GPIO4/RXD: R309.1
- new net GPIO5/TXD: R304.1
- no-connect marks 14 -> 8
Other:
- note removed: "ABM3-8.000MHZ-B4Y-T"
- moved on the sheet: C305, C306, U201D, U201F, U201G
