File: Electrique/SoM_V2/SoM_V2/Sortie.kicad_sch (KiCad schematic)
At the start: 8 parts, among them U501 PCA9633DP1

Commit message: stinky kicad
Changed lines of the file:
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@@
 		(dnp no)
 		(property "Reference" "J201"
-			(at 219.71 24.13 0)
+			(at 219.964 21.59 0)
 			(effects
 				(font

Commit message: push fix ???
Parts:
- removed J201: ~, connecteur_M2_key_E:NGFF_E, symbol connecteur_m2_key_E:connecteur_SOM_ESP32
- added U1: ~, connecteur_M2_key_E:NGFF_E, symbol connecteur_m2_key_E:connecteur_SOM_ESP32_V2
- renumbered C501 to C401, C502 to C402, C503 to C403, D501 to D401, R501 to R401, R502 to R402, U501 to U401
Connections:
- net GPIO15: now also U1.40 (GPIO15)
- net GPIO16: now also U1.41 (GPIO16)
- net GPIO26: now also U1.42 (GPIO26)
- net GPIO33: now also U1.43 (GPIO33)
- net GPIO34: now also U1.44 (GPIO34)
- net GPIO38_ADDRESSABLE_LED: now also U1.6 (GPIO38&LED)
- net GPIO45: now also U1.52 (GPIO45)
- net GPIO46: now also U1.53 (GPIO46)
- net GPIO48/CAN_INT: now also U1.36 (GPIO48)
- net at U401.1 (PWM1): now also U1.64 (PWM_1_PCA)
- net at U401.2 (PWM2): now also U1.66 (PWM_2_PCA)
- net at U401.3 (PWM3): now also U1.68 (PWM_3_PCA)
- net at U401.4 (PWM4): now also U1.70 (PWM_4_PCA)
- new net RESET_OTHERS: U1.34 (RST_OTHER)
- no-connect marks 3 -> 1
Other:
- note removed: "REFCLK n'est pas un feature En gros le SDK de ESP-IDF ne le supporte pas???? https://www.esp32.com/viewtopic.php?t=3011 à vérifier"

Commit message: push v2.2
Parts:
- R401, R402: value 10k -> 1k
- renumbered U1 to U201
Connections:
- net RESET_OTHERS: no longer names the net of U201.34 (RST_OTHER)
- no-connect marks 1 -> 2
Changed lines of the file:
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@@
 		(at 254 62.23)
+	)
+	(no_connect
+		(at 236.22 31.75)
 	)
 	(wire
@@
 				)
 				(justify right)
-				(hide yes)
-			)
-		)
-	)
-	(global_label "RESET_OTHERS"
-		(shape input)
-		(at 236.22 31.75 0)
-		(fields_autoplaced yes)
-		(effects
-			(font
-				(size 1.27 1.27)
-			)
-			(justify left)
-		)
-		(property "Intersheetrefs" "${INTERSHEET_REFS}"
-			(at 253.175 31.75 0)
-			(effects
-				(font
-					(size 1.27 1.27)
-				)
-				(justify left)
 				(hide yes)
 			)
@@
 		(on_board yes)
 		(dnp no)
-		(property "Reference" "U1"
+		(property "Reference" "U201"
 			(at 220.98 21.59 0)
 			(effects
@@
 		(instances
 			(project "SoM_V2"
-				(path "/ecd44d9a-8113-48e2-a5bb-0de07ce8b9ce/8e20c774-e159-4c82-b251-7add9faa2a44"
-					(reference "U1")
-					(unit 10)
-				)
 				(path "/ecd44d9a-8113-48e2-a5bb-0de07ce8b9ce/fc7293f1-5a36-4fea-b330-faa9d597a61e"
 					(reference "U201")
@@
 			)
 		)
-		(property "Value" "10k"
+		(property "Value" "1k"
 			(at 72.39 21.59 0)
 			(effects
@@
 			)
 		)
-		(property "Value" "10k"
+		(property "Value" "1k"
 			(at 64.77 21.59 0)
 			(effects
@@
 		(on_board yes)
 		(dnp no)
-		(property "Reference" "U1"
+		(property "Reference" "U201"
 			(at 115.57 21.59 0)
 			(effects
@@
 		(instances
 			(project "SoM_V2"
-				(path "/ecd44d9a-8113-48e2-a5bb-0de07ce8b9ce/8e20c774-e159-4c82-b251-7add9faa2a44"
-					(reference "U1")
-					(unit 9)
-				)
 				(path "/ecd44d9a-8113-48e2-a5bb-0de07ce8b9ce/fc7293f1-5a36-4fea-b330-faa9d597a61e"
 					(reference "U201")
