File: Electrique/SoM_V2/Alimentation.kicad_sch (KiCad schematic)
At the start: 3 parts

Commit message: Clean up schema et PCB
Connections:
- net +3V3: now also D201.2 (A); no longer D201.1 (K)
- net at R201.1: now also D201.1 (K); no longer D201.2 (A)
Other:
- moved on the sheet: D201
Changed lines of the file:
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@@
 	(symbol
 		(lib_id "Device:LED")
-		(at 103.505 76.835 270)
+		(at 103.505 76.835 90)
 		(unit 1)
 		(exclude_from_sim no)
@@
 		(fields_autoplaced yes)
 		(property "Reference" "D201"
-			(at 106.68 73.9774 90)
+			(at 106.68 77.1524 90)
 			(effects
 				(font
 					(size 1.27 1.27)
 				)
-				(justify left)
+				(justify right)
 			)
 		)
 		(property "Value" "GREEN"
-			(at 106.68 76.5174 90)
+			(at 106.68 79.6924 90)
 			(effects
 				(font
 					(size 1.27 1.27)
 				)
-				(justify left)
+				(justify right)
 			)
 		)
