File: Electrique/SoM_V2/ESP32.kicad_sch (KiCad schematic)
At the start: 12 parts, among them Q501 MBT3904DW1T1G, SW501 SW_BOOT, SW502 SW_CHIP_EN, U501 ESP32-S3-MINI-1U

Commit message: Clean up schema et PCB
Other:
- note added: "Circuit de reset et de prog avec boutons"
- note added: "Module ESP32-S3-MINI-U1"
Changed lines of the file:
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@@
+		)
+	)
+	(rectangle
+		(start 200.66 13.97)
+		(end 281.94 124.46)
+		(stroke
+			(width 1)
+			(type default)
+		)
+		(fill
+			(type none)
+		)
+	)
+	(rectangle
+		(start 12.7 12.7)
+		(end 136.144 100.33)
+		(stroke
+			(width 1)
+			(type default)
+		)
+		(fill
+			(type none)
+		)
+	)
+	(text "Module ESP32-S3-MINI-U1\n"
+		(exclude_from_sim no)
+		(at 13.716 99.314 0)
+		(effects
+			(font
+				(size 1.27 1.27)
+			)
+			(justify left)
+		)
+	)
+	(text "Circuit de reset et de prog avec boutons"
+		(exclude_from_sim no)
+		(at 201.168 122.936 0)
+		(effects
+			(font
+				(size 1.27 1.27)
+			)
+			(justify left)
 		)
 	)
