File: Electrique/MOBO_V2/MOBO_V2.kicad_pcb (KiCad board)
At the start: 4 copper layers, 39.4 x 98.5 mm, 46 parts, among them J1 Gauche, J2 Droite, J301 USB_C_UART, J302 USB_C_DEBUG, J307 I2C_0_0, J308 I2C_0_1, J309 I2C_1_0, J310 I2C_1_1, Q1 AO3401A, U2 TPS562242DRLR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

Commit message: verified by frank
Routing:
- net Net-(U2-EN): track 20.9 -> 20.3 mm
